File: PCB_Principal/ISPEL-CAD_v1.kicad_pcb (KiCad board)
At the start: 2 copper layers, 130 x 160 mm, 184 parts, among them J1 Vin, J10 GND_NUCLEO, J11 CN7_NUCLEO, J12 CN10_NUCLEO, J13 GND_NUCLEO, J14 E1, J15 S1, J16 E2, J17 S2, J18 FRENTE, J19 PRUEBA_5V, J2 V7, J3 TEMP, J4 VREG, J5 V5, J6 GND_NUCLEO, J7 CN8_NUCLEO, J8 CN9_NUCLEO, J9 GND_NUCLEO, Q201 BC807, Q202 BC559C, Q203 BC549C, Q204 BC549C, Q205 BC559C, Q206 2SD882, Q207 2SB772, Q251 BC807, Q252 BC559C, Q253 BC549C, Q254 BC549C, Q255 BC559C, Q256 2SD882, Q257 2SB772, U1 LM350_TO220, U101 TL071, U151 TL071, U2 LM350_TO220, U201 LM318, U251 LM318, U3 LM337_TO220, U301 TLV3501AID, U4 LM1117DT-5.0, U5 TL431DBZ

Commit message: Revisión 1. Con prototipo ISPEL Beta 2024 en fase de prueba.
Parts:
- C102, C152: value 3.3pF -> 5pF
- C5, C6, C7, C8: value 220nF -> 1uF
- R14: value 0 -> 0.1
- R15, RT1, RT2, RT3, RT4, RT5: value 1 -> 0.1
- R216, R217, R266, R267: value 1M -> CAL
- U101, U151: value TL071 -> CA3140
Changed lines of the file:
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@@
 			)
 		)
-		(property "Value" "1"
+		(property "Value" "0.1"
 			(at 0 1.82 90)
 			(layer "F.Fab")
@@
 			)
 		)
-		(property "Value" "3.3pF"
+		(property "Value" "5pF"
 			(at -0.155 -1.8 0)
 			(layer "F.Fab")
@@
 			)
 		)
-		(property "Value" "1"
+		(property "Value" "0.1"
 			(at 0 1.82 90)
 			(layer "F.Fab")
@@
 			)
 		)
-		(property "Value" "0"
+		(property "Value" "0.1"
 			(at 0 1.82 0)
 			(layer "F.Fab")
@@
 			)
 		)
-		(property "Value" "3.3pF"
+		(property "Value" "5pF"
 			(at -0.1625 -1.95 0)
 			(layer "F.Fab")
@@
 			)
 		)
-		(property "Value" "1"
+		(property "Value" "0.1"
 			(at 0 1.82 0)
 			(layer "F.Fab")
@@
 			)
 		)
-		(property "Value" "220nF"
+		(property "Value" "1uF"
 			(at 0 1.85 0)
 			(layer "F.Fab")
@@
 			)
 		)
-		(property "Value" "1"
+		(property "Value" "0.1"
 			(at 0 1.82 0)
 			(layer "F.Fab")
@@
 			)
 		)
-		(property "Value" "TL071"
+		(property "Value" "CA3140"
 			(at 3.81 11.475 0)
 			(layer "F.Fab")
@@
 			)
 		)
-		(property "Datasheet" "http://www.ti.com/lit/ds/symlink/tl071.pdf"
+		(property "Datasheet" "https://www.renesas.com/en/document/dst/ca3140-ca3140a-datasheet?r=505296"
 			(at 0 0 0)
 			(unlocked yes)
@@
 			)
 		)
-		(property "Description" "Single Low-Noise JFET-Input Operational Amplifiers, DIP-8/SOIC-8"
+		(property "Description" "4.5MHz, BiMOS Operational Amplifier with MOSFET Input/Bipolar Output"
 			(at 0 0 0)
 			(unlocked yes)
@@
 			)
 		)
-		(property "Value" "1"
+		(property "Value" "0.1"
 			(at 0 1.82 0)
 			(layer "F.Fab")
@@
 			)
 		)
-		(property "Value" "TL071"
+		(property "Value" "CA3140"
 			(at 3.81 11.475 0)
 			(layer "F.Fab")
@@
 			)
 		)
-		(property "Datasheet" "http://www.ti.com/lit/ds/symlink/tl071.pdf"
+		(property "Datasheet" "https://www.renesas.com/en/document/dst/ca3140-ca3140a-datasheet?r=505296"
 			(at 0 0 0)
 			(unlocked yes)
@@
 			)
 		)
-		(property "Description" "Single Low-Noise JFET-Input Operational Amplifiers, DIP-8/SOIC-8"
+		(property "Description" "4.5MHz, BiMOS Operational Amplifier with MOSFET Input/Bipolar Output"
 			(at 0 0 0)
 			(unlocked yes)
@@
 			)
 		)
-		(property "Value" "1"
+		(property "Value" "0.1"
 			(at 0 1.82 90)
 			(layer "F.Fab")
@@
 			)
 		)
-		(property "Value" "220nF"
+		(property "Value" "1uF"
 			(at 0.125 1.575 0)
 			(layer "B.Fab")
@@
 			)
 		)
-		(property "Value" "220nF"
+		(property "Value" "1uF"
 			(at 0.075 1.6 0)
 			(layer "B.Fab")
@@
 			)
 		)
-		(property "Value" "1M"
+		(property "Value" "CAL"
 			(at 0 -1.82 0)
 			(layer "B.Fab")
@@
 			)
 		)
-		(property "Value" "1M"
+		(property "Value" "CAL"
 			(at 0 -1.82 0)
 			(layer "B.Fab")
@@
 			)
 		)
-		(property "Value" "1M"
+		(property "Value" "CAL"
 			(at 0 -1.82 0)
 			(layer "B.Fab")
@@
 			)
 		)
-		(property "Value" "220nF"
+		(property "Value" "1uF"
 			(at 0 -1.85 0)
 			(layer "B.Fab")
@@
 			)
 		)
-		(property "Value" "1M"
+		(property "Value" "CAL"
 			(at 0 -1.82 0)
 			(layer "B.Fab")
